File: LCC_Interface.kicad_pcb (KiCad board)
At the start: 2 copper layers, 60 x 50 mm, 18 parts, among them J1 LCC RJ45, J2 LCC RJ45, J3 MCU INTERFACE, U1 TCAN332DR

Commit message: Add Rev C: diagnostic LEDs/test points, RJ45 models, Gerbers
Parts:
- added D2: LED, LED_SMD:LED_0805_2012Metric_Pad1.15x1.40mm_HandSolder, F.Cu at (19.5, 41.0)
- added D3: LED, LED_SMD:LED_0805_2012Metric_Pad1.15x1.40mm_HandSolder, F.Cu at (28.5, 41.0)
- added D4: LED, LED_SMD:LED_0805_2012Metric_Pad1.15x1.40mm_HandSolder, F.Cu at (37.5, 41.0)
- added R4: 1k, Resistor_SMD:R_0805_2012Metric_Pad1.20x1.40mm_HandSolder, F.Cu at (15.0, 41.0)
- added R5: 1k, Resistor_SMD:R_0805_2012Metric_Pad1.20x1.40mm_HandSolder, F.Cu at (24.0, 41.0)
- added R6: 1k, Resistor_SMD:R_0805_2012Metric_Pad1.20x1.40mm_HandSolder, F.Cu at (33.0, 41.0)
- added TP4: TP, TestPoint:TestPoint_THTPad_D1.5mm_Drill0.7mm, F.Cu at (53.0, 12.0)
- added TP5: TP, TestPoint:TestPoint_THTPad_D1.5mm_Drill0.7mm, F.Cu at (53.0, 16.0)
- added TP6: TP, TestPoint:TestPoint_THTPad_D1.5mm_Drill0.7mm, F.Cu at (53.0, 20.0)
Routing:
- net /+3V3: track 16.4 -> 106.5 mm, vias 0 -> 1
- net /CAN_TX: track 21.3 -> 87.5 mm
- net /CAN_RX: track 17.4 -> 79.0 mm
- net /LED_PWR: track 0.00 -> 8.05 mm
- net /CAN_H: track 74.3 -> 81.4 mm
- net /LED_TX: track 0.00 -> 5.90 mm
- net /LED_RX: track 0.00 -> 5.38 mm
- net /CAN_GND: track 138.1 -> 142.6 mm, vias 0 -> 1
Other:
- board text added: "+3V3"
- board text added: "CAN_RX"
- board text added: "CAN_TX"
- board text added: "LCC / CAN INTERFACE Rev C"
- board text added: "PWR"
- board text removed: "LCC / CAN INTERFACE Rev B"
