File: LCC_Interface.kicad_sch (KiCad schematic)
At the start: 11 parts, among them J1 LCC RJ45, J2 LCC RJ45, J3 MCU INTERFACE, U1 TCAN332DR

Commit message: Add Rev C: diagnostic LEDs/test points, RJ45 models, Gerbers
Parts:
- added D2, D3, D4: LED, LED_SMD:LED_0805_2012Metric_Pad1.15x1.40mm_HandSolder, symbol LCC:LED
- added R4, R5, R6: 1k, Resistor_SMD:R_0805_2012Metric_Pad1.20x1.40mm_HandSolder, symbol LCC:R
Connections:
- net +3V3: now also R4.1, R5.1, R6.1
- net CAN_GND: now also D2.1 (K)
- net CAN_RX: now also D4.1 (K)
- net CAN_TX: now also D3.1 (K)
- new net LED_PWR: D2.2 (A), R4.2
- new net LED_RX: D4.2 (A), R6.2
- new net LED_TX: D3.2 (A), R5.2
Other:
- note added: "Rev C: passive diagnostics - D2 power LED (via R4), D3 TX LED (via R5), D4 RX LED (via R6), all 1k; probe pads TP4-6 (board-only) on +3V3/CAN_TX/CAN_RX."
- note added: "Universal LCC / CAN Interface Rev C"
- note removed: "Universal LCC / CAN Interface Rev B"
- company: LCC Interface - Rev B -> LCC Interface - Rev C
Changed lines of the file:
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@@
  (generator_version "8.0")
  (paper "A4")
- (title_block (title "Universal LCC CAN Interface") (date "2026-08-30") (rev "B") (company "LCC Interface - Rev B"))
+ (title_block (title "Universal LCC CAN Interface") (date "2026-08-30") (rev "C") (company "LCC Interface - Rev C"))
  (label "CAN_TX" (at 109.84 89.92 180) (effects (font (size 1.27 1.27))))
 (label "CAN_RX" (at 109.84 100.08 180) (effects (font (size 1.27 1.27))))
@@
 (label "CAN_L" (at 133.65 97.54 0) (effects (font (size 1.0 1.0))))
 (label "CAN_GND" (at 140 101.35 270) (effects (font (size 1.0 1.0))))
- (text "Universal LCC / CAN Interface Rev B" (exclude_from_sim no) (at 95 40 0) (effects (font (size 1.8 1.8))))
+ (text "Universal LCC / CAN Interface Rev C" (exclude_from_sim no) (at 95 40 0) (effects (font (size 1.8 1.8))))
+(text "Rev C: passive diagnostics - D2 power LED (via R4), D3 TX LED (via R5), D4 RX LED (via R6), all 1k; probe pads TP4-6 (board-only) on +3V3/CAN_TX/CAN_RX." (exclude_from_sim no) (at 100 160 0) (effects (font (size 1.0 1.0))))
 (text "RJ45 pin 3 CAN_GND and pin 6 share CAN_GND net; shell (SH) also on CAN_GND" (exclude_from_sim no) (at 100 145 0) (effects (font (size 1.0 1.0))))
 (text "PWR_NEG remains separate. Bus power is pass-through only. Local ground = CAN_GND." (exclude_from_sim no) (at 100 150 0) (effects (font (size 1.0 1.0))))
@@
  (instances (project "LCC_Interface" (path "/bf935f1b-10d6-47c4-8946-ddf1a2732d35" (reference "JP1") (unit 1))))
 )
+ (label "+3V3" (at 76.19 165 180) (effects (font (size 1.27 1.27))))
+(label "LED_PWR" (at 83.81 165 0) (effects (font (size 1.27 1.27))))
+(label "CAN_GND" (at 91.19 165 180) (effects (font (size 1.27 1.27))))
+(label "LED_PWR" (at 98.81 165 0) (effects (font (size 1.27 1.27))))
+(label "+3V3" (at 76.19 175 180) (effects (font (size 1.27 1.27))))
+(label "LED_TX" (at 83.81 175 0) (effects (font (size 1.27 1.27))))
+(label "CAN_TX" (at 91.19 175 180) (effects (font (size 1.27 1.27))))
+(label "LED_TX" (at 98.81 175 0) (effects (font (size 1.27 1.27))))
+(label "+3V3" (at 76.19 185 180) (effects (font (size 1.27 1.27))))
+(label "LED_RX" (at 83.81 185 0) (effects (font (size 1.27 1.27))))
+(label "CAN_RX" (at 91.19 185 180) (effects (font (size 1.27 1.27))))
+(label "LED_RX" (at 98.81 185 0) (effects (font (size 1.27 1.27))))
+ (symbol (lib_id "LCC:R") (at 80 165 0) (unit 1) (in_bom yes) (on_board yes) (dnp no)
+ (property "Reference" "R4" (at 80 161.5 0) (effects (font (size 1.27 1.27))))
+ (property "Value" "1k" (at 80 168.5 0) (effects (font (size 1.27 1.27))))
+ (property "Footprint" "Resistor_SMD:R_0805_2012Metric_Pad1.20x1.40mm_HandSolder" (at 80 165 0) (effects (font (size 1.27 1.27)) hide))
+ (property "Datasheet" "" (at 80 165 0) (effects (font (size 1.27 1.27)) hide))
+ (pin "1")
+(pin "2")
+ (instances (project "LCC_Interface" (path "/bf935f1b-10d6-47c4-8946-ddf1a2732d35" (reference "R4") (unit 1))))
+)
+(symbol (lib_id "LCC:LED") (at 95 165 0) (unit 1) (in_bom yes) (on_board yes) (dnp no)
+ (property "Reference" "D2" (at 95 161.5 0) (effects (font (size 1.27 1.27))))
+ (property "Value" "LED" (at 95 168.5 0) (effects (font (size 1.27 1.27))))
+ (property "Footprint" "LED_SMD:LED_0805_2012Metric_Pad1.15x1.40mm_HandSolder" (at 95 165 0) (effects (font (size 1.27 1.27)) hide))
+ (property "Datasheet" "" (at 95 165 0) (effects (font (size 1.27 1.27)) hide))
+ (pin "1")
+(pin "2")
+ (instances (project "LCC_Interface" (path "/bf935f1b-10d6-47c4-8946-ddf1a2732d35" (reference "D2") (unit 1))))
+)
+(symbol (lib_id "LCC:R") (at 80 175 0) (unit 1) (in_bom yes) (on_board yes) (dnp no)
+ (property "Reference" "R5" (at 80 171.5 0) (effects (font (size 1.27 1.27))))
+ (property "Value" "1k" (at 80 178.5 0) (effects (font (size 1.27 1.27))))
+ (property "Footprint" "Resistor_SMD:R_0805_2012Metric_Pad1.20x1.40mm_HandSolder" (at 80 175 0) (effects (font (size 1.27 1.27)) hide))
+ (property "Datasheet" "" (at 80 175 0) (effects (font (size 1.27 1.27)) hide))
+ (pin "1")
+(pin "2")
+ (instances (project "LCC_Interface" (path "/bf935f1b-10d6-47c4-8946-ddf1a2732d35" (reference "R5") (unit 1))))
+)
+(symbol (lib_id "LCC:LED") (at 95 175 0) (unit 1) (in_bom yes) (on_board yes) (dnp no)
+ (property "Reference" "D3" (at 95 171.5 0) (effects (font (size 1.27 1.27))))
+ (property "Value" "LED" (at 95 178.5 0) (effects (font (size 1.27 1.27))))
+ (property "Footprint" "LED_SMD:LED_0805_2012Metric_Pad1.15x1.40mm_HandSolder" (at 95 175 0) (effects (font (size 1.27 1.27)) hide))
+ (property "Datasheet" "" (at 95 175 0) (effects (font (size 1.27 1.27)) hide))
+ (pin "1")
+(pin "2")
+ (instances (project "LCC_Interface" (path "/bf935f1b-10d6-47c4-8946-ddf1a2732d35" (reference "D3") (unit 1))))
+)
+(symbol (lib_id "LCC:R") (at 80 185 0) (unit 1) (in_bom yes) (on_board yes) (dnp no)
+ (property "Reference" "R6" (at 80 181.5 0) (effects (font (size 1.27 1.27))))
+ (property "Value" "1k" (at 80 188.5 0) (effects (font (size 1.27 1.27))))
+ (property "Footprint" "Resistor_SMD:R_0805_2012Metric_Pad1.20x1.40mm_HandSolder" (at 80 185 0) (effects (font (size 1.27 1.27)) hide))
+ (property "Datasheet" "" (at 80 185 0) (effects (font (size 1.27 1.27)) hide))
+ (pin "1")
+(pin "2")
+ (instances (project "LCC_Interface" (path "/bf935f1b-10d6-47c4-8946-ddf1a2732d35" (reference "R6") (unit 1))))
+)
+(symbol (lib_id "LCC:LED") (at 95 185 0) (unit 1) (in_bom yes) (on_board yes) (dnp no)
+ (property "Reference" "D4" (at 95 181.5 0) (effects (font (size 1.27 1.27))))
+ (property "Value" "LED" (at 95 188.5 0) (effects (font (size 1.27 1.27))))
+ (property "Footprint" "LED_SMD:LED_0805_2012Metric_Pad1.15x1.40mm_HandSolder" (at 95 185 0) (effects (font (size 1.27 1.27)) hide))
+ (property "Datasheet" "" (at 95 185 0) (effects (font (size 1.27 1.27)) hide))
+ (pin "1")
+(pin "2")
+ (instances (project "LCC_Interface" (path "/bf935f1b-10d6-47c4-8946-ddf1a2732d35" (reference "D4") (unit 1))))
+)
  (sheet_instances (path "/" (page "1")))
